File: circuit/Barometer/Barometer.kicad_pcb (KiCad board)
At the start: 2 copper layers, 0 parts

Commit message: 回路図&PCBを追加
Parts:
- added C1: 0.1u, Capacitor_SMD:C_0603_1608Metric_Pad1.08x0.95mm_HandSolder, B.Cu at (114.0, 69.1)
- added C2: 0.1u, Capacitor_SMD:C_0603_1608Metric_Pad1.08x0.95mm_HandSolder, F.Cu at (107.7, 71.3)
- added C3: 1.0u, Capacitor_SMD:C_0603_1608Metric_Pad1.08x0.95mm_HandSolder, F.Cu at (103.8, 68.5)
- added D1: LED, Diode_SMD:D_0603_1608Metric_Pad1.05x0.95mm_HandSolder, F.Cu at (115.5, 61.2)
- added G***: LOGO, NABA:AIOLIA, F.Cu at (107.0, 60.4)
- added J1: Conn_01x06_Female, Connector_PinSocket_2.54mm:PinSocket_1x06_P2.54mm_Vertical, F.Cu at (95.6, 73.2)
- added J2: Conn_01x04_Socket, Connector:NS-Tech_Grove_1x04_P2mm_Vertical, F.Cu at (106.2, 76.7)
- added J3: Conn_01x02, Connector_JST:JST_PH_B2B-PH-K_1x02_P2.00mm_Vertical, F.Cu at (113.1, 76.5)
- added R1: 10k, Resistor_SMD:R_0603_1608Metric_Pad0.98x0.95mm_HandSolder, F.Cu at (102.1, 65.3)
- added R2: 10k, Resistor_SMD:R_0603_1608Metric_Pad0.98x0.95mm_HandSolder, F.Cu at (103.7, 65.3)
- added R3: 200, Resistor_SMD:R_0603_1608Metric_Pad0.98x0.95mm_HandSolder, F.Cu at (115.5, 64.7)
- added SW1: SW_Slide, AIOLIA:SW_Slide, F.Cu at (113.1, 70.0)
- added U1: TWE-L-WX, RF_Module:MonoWireless_TWE-L-WX, B.Cu at (105.3, 67.5)
- added U2: ~, AIOLIA:SOT95P280X130-5N, F.Cu at (104.7, 71.4)
Routing:
- net GND: track 0.00 -> 41.9 mm, vias 0 -> 36
- net +3V3: track 0.00 -> 37.5 mm, vias 0 -> 1
- net Net-(J1-Pin_3): track 0.00 -> 28.0 mm
- net Net-(J1-Pin_2): track 0.00 -> 24.5 mm
- net VCC: track 0.00 -> 18.8 mm, vias 0 -> 2
- net Net-(J1-Pin_4): track 0.00 -> 18.1 mm, vias 0 -> 1
- net Net-(J1-Pin_5): track 0.00 -> 9.48 mm, vias 0 -> 1
- net Net-(J3-Pin_1): track 0.00 -> 8.60 mm
- net SDA: track 0.00 -> 8.46 mm
- net Net-(U1-ADC1/AI1): track 0.00 -> 5.16 mm, vias 0 -> 1
- net SCL: track 0.00 -> 4.17 mm
- net LED1: track 0.00 -> 3.48 mm, vias 0 -> 1
- net Net-(D1-A): track 0.00 -> 1.71 mm
- added copper zone on B.Cu, net GND
- added copper zone on F.Cu, net GND
Other:
- board outline added: 24.4 x 21.6 mm
- board text added: "3V3"
- board text added: "GND"
- board text added: "PRG"
- board text added: "RST"
- board text added: "RXD"
- board text added: "SCL"
- board text added: "SDA"
- board text added: "TXD"
- board text added: "VCC"
