File: circuit/Barometer/Barometer.kicad_sch (KiCad schematic)
At the start: 0 parts

Commit message: initial commit
Other:
- title: Template -> Barometer
Changed lines of the file:
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@@
 	(paper "A4")
 	(title_block
-		(title "Template")
+		(title "Barometer")
 		(rev "0.0")
 		(company "AIOLIA")

Commit message: 回路図&PCBを追加
Parts:
- added C1, C2: 0.1u, Capacitor_SMD:C_0603_1608Metric_Pad1.08x0.95mm_HandSolder, symbol Device:C
- added C3: 1.0u, Capacitor_SMD:C_0603_1608Metric_Pad1.08x0.95mm_HandSolder, symbol Device:C
- added D1: LED, Diode_SMD:D_0603_1608Metric_Pad1.05x0.95mm_HandSolder, symbol Device:LED
- added J1: Conn_01x06_Female, Connector_PinSocket_2.54mm:PinSocket_1x06_P2.54mm_Vertical, symbol Connector:Conn_01x06_Female
- added J2: Conn_01x04_Socket, Connector:NS-Tech_Grove_1x04_P2mm_Vertical, symbol Connector:Conn_01x04_Socket
- added J3: Conn_01x02, Connector_JST:JST_PH_B2B-PH-K_1x02_P2.00mm_Vertical, symbol Connector_Generic:Conn_01x02
- added R1, R2: 10k, Resistor_SMD:R_0603_1608Metric_Pad0.98x0.95mm_HandSolder, symbol Device:R
- added R3: 200, Resistor_SMD:R_0603_1608Metric_Pad0.98x0.95mm_HandSolder, symbol Device:R
- added SW1: SW_Slide, AIOLIA:SW_Slide, symbol AIOLIA:SW_Slide
- added U1: TWE-L-WX, RF_Module:MonoWireless_TWE-L-WX, symbol RF_ZigBee:TWE-L-WX
- added U2: ~, AIOLIA:SOT95P280X130-5N, symbol AIOLIA:NJM2866F33
Connections:
- new net: D1.2 (A), R3.2
- new net: R1.2, R2.2, U1.23 (ADC1/AI1)
- new net: J1.3 (Pin_3), U1.2 (DO1/PWM3)
- new net: J1.5 (Pin_5), U1.21 (~{RESET})
- new net: J1.2 (Pin_2), U1.8 (DIO6/TX)
- new net: J1.4 (Pin_4), U1.9 (DIO7/RX)
- new net: J3.1 (Pin_1), SW1.2 (B), SW1.5 (B)
- new net +3V3: C1.1, C3.2, J1.6 (Pin_6), J2.3 (Pin_3), U1.5 (VCC), U2.5 (Vout)
- new net GND: C1.2, C2.2, C3.1, D1.1 (K), J1.1 (Pin_1), J2.4 (Pin_4), J3.2 (Pin_2), R1.1, U1.20 (GND), U1.22 (ADC2/AI3), U1.24 (DIO0/AI2), U1.25 (DIO1/AI4), U1.28 (GND), U1.30 (GND), U1.31 (GND), U1.32 (GND), U2.2 (GND)
- new net LED1: R3.1, U1.3 (DIO18/DO1)
- new net SCL: J2.1 (Pin_1), U1.14 (DIO14/SCL)
- new net SDA: J2.2 (Pin_2), U1.17 (DIO15/SDA)
- new net VCC: C2.1, R2.1, SW1.1 (A), SW1.6 (C), U2.1 (Vin), U2.3 (CONTROL)
- no-connect marks 0 -> 16
Other:
- note added: "TWELITE"
- company: AIOLIA -> NABA
